File: trailer-power-controller/trailer-power-controller.kicad_pcb (KiCad board)
At the start: 2 copper layers, 106.4 x 52.8 mm, 83 parts, among them J1 Anderson_two_redblack_src, J2 USB_B_Micro, J3 Conn_01x02, J4 Conn_01x03, J5 Conn_01x03, J6 Conn_01x02, J7 Anderson_two_redblack_sink, Q1 Q_NPN_BEC, Q2 Q_NPN_BEC, Q3 AO3400A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

Commit message: trailer-power-controller hardware v1.0
Parts:
- added F1: 1A Polyfuse, Fuse:Fuse_1206_3216Metric_Pad1.42x1.75mm_HandSolder, F.Cu at (131.7, 103.0)
- added J9: Conn_01x02, Connector_PinHeader_2.54mm:PinHeader_1x02_P2.54mm_Vertical, F.Cu at (61.8, 59.4)
- added R27: 470, Resistor_SMD:R_0402_1005Metric, F.Cu at (125.2, 101.3)
- moved C7 15.9 mm to (111.7, 96.2), turned to 90 degrees
- moved R9 13.6 mm to (111.2, 97.7)
- moved R4 12.4 mm to (116.2, 95.4), turned to 180 degrees
- moved D1 8.87 mm to (127.2, 103.7)
- moved R5 7.92 mm to (116.2, 100.0)
- moved C16 7.36 mm to (102.4, 106.0), turned to 90 degrees
- moved D4 7.26 mm to (138.4, 80.9)
- moved R6 7.26 mm to (135.9, 80.9)
- moved C11 7.11 mm to (90.3, 74.8), turned to 180 degrees
- moved D3 7.01 mm to (96.5, 86.8)
- moved R2 7.01 mm to (99.1, 86.8)
- moved Q2 6.82 mm to (118.2, 97.7), turned to 180 degrees
- moved C2 6.50 mm to (122.6, 96.6)
- moved U2 6.50 mm to (128.4, 96.5)
- moved R1 6.50 mm to (126.5, 101.3)
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Connections:
- net /USB_DM renamed /USB_DN
- J2 pad 1: Net-(D1-Pad2) -> Net-(F1-Pad2)
- U1 pad 10: unconnected-(U1-Pad10) -> /BUZZER
- U1 pad 11: unconnected-(U1-Pad11) -> /TEMP_INTERAL
- U1 pad 12: unconnected-(U1-Pad12) -> /TEMP_EXTERNAL
- U1 pad 13: /RELAY_EN -> unconnected-(U1-Pad13)
- U1 pad 27: /TEMP_INTERNAL -> unconnected-(U1-Pad27)
- U1 pad 28: /TEMP_EXTERNAL -> unconnected-(U1-Pad28)
- U1 pad 34: /USB_TX -> Net-(U1-Pad34)
- U1 pad 36: unconnected-(U1-Pad36) -> /RELAY_EN
Routing:
- net GND: track 0.00 -> 258.9 mm, vias 0 -> 63
- net +3V3: track 0.00 -> 189.8 mm, vias 0 -> 9
- net /VEHICLE+: track 0.00 -> 180.5 mm, vias 0 -> 5
- net /BATTERY+: track 0.00 -> 70.0 mm, vias 0 -> 1
- net /RELAY_EN: track 0.00 -> 67.3 mm, vias 0 -> 2
- net /TEMP_AUX: track 0.00 -> 56.9 mm, vias 0 -> 2
- net Net-(C18-Pad1): track 0.00 -> 50.9 mm, vias 0 -> 2
- net /LOAD_SENSE: track 0.00 -> 48.7 mm, vias 0 -> 2
- net /EN: track 0.00 -> 41.1 mm, vias 0 -> 2
- net /CHARGE_EN: track 0.00 -> 33.9 mm, vias 0 -> 2
- net Net-(R1-Pad1): track 0.00 -> 31.8 mm, vias 0 -> 2
- net /BUZZER: track 0.00 -> 31.7 mm, vias 0 -> 2
- net Net-(U1-Pad34): track 0.00 -> 30.0 mm, vias 0 -> 2
- net /TEMP_EXTERNAL: track 0.00 -> 26.4 mm, vias 0 -> 2
- net /VEHICLE_SENSE: track 0.00 -> 21.0 mm
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- added copper zone on B.Cu, net GND
- added copper zone on F.Cu, net GND
Other:
- board size 106.4 x 52.8 mm -> 94.3 x 52.8 mm
- board text added: "3V3"
- board text added: "AUX"
- board text added: "BATTERY"
- board text added: "BREAKER"
- board text added: "EXT"
- board text added: "GND"
- board text added: "IN"
- board text added: "OUT"
- board text added: "RELAY"
- board text added: "RESET"
- board text added: "SW1"
- board text added: "SW2"
- board text added: "TRAILER"
- board text added: "trailer-power-controller v1.0"

Commit message: Pre-fab hardware v1.0 fixes
Parts:
- added D12: D, Diode_SMD:D_SOD-323, F.Cu at (96.3, 95.3)
Routing:
- net /BATTERY+: track 70.0 -> 76.8 mm
