File: trailer-power-controller/trailer-power-controller.kicad_sch (KiCad schematic)
At the start: 83 parts, among them J1 Anderson_two_redblack_src, J2 USB_B_Micro, J3 Conn_01x02, J4 Conn_01x03, J5 Conn_01x03, J6 Conn_01x02, J7 Anderson_two_redblack_sink, Q1 Q_NPN_BEC, Q2 Q_NPN_BEC, Q3 AO3400A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

Commit message: trailer-power-controller hardware v1.0
Parts:
- added F1: 1A Polyfuse, Fuse:Fuse_1206_3216Metric_Pad1.42x1.75mm_HandSolder, symbol Device:Polyfuse
- added J9: Conn_01x02, Connector_PinHeader_2.54mm:PinHeader_1x02_P2.54mm_Vertical, symbol Connector_Generic:Conn_01x02
- added R27: 470, Resistor_SMD:R_0402_1005Metric, symbol Device:R
Connections:
- net +3V3: now also J9.2 (Pin_2)
- net BUZZER: now also U1.10 (IO25)
- net GND: now also J9.1 (Pin_1)
- net RELAY_EN: now also U1.36 (IO22); no longer U1.13 (IO14)
- net TEMP_EXTERNAL: now also U1.12 (IO27); no longer U1.28 (IO17)
- net TEMP_INTERAL: now also U1.11 (IO26)
- net USB_TX: now also R27.2; no longer U1.34 (RXD0/IO3)
- net at D1.2 (A): now also F1.1; no longer J2.1 (VBUS)
- net TEMP_INTERNAL: no longer names the net of U1.27 (IO16)
- net USB_DM renamed USB_DN
- new net: R27.1, U1.34 (RXD0/IO3)
- new net: F1.2, J2.1 (VBUS)
- no-connect marks 23 -> 22
Other:
- moved on the sheet: D1, R1

Commit message: Pre-fab hardware v1.0 fixes
Parts:
- added D12: D, Diode_SMD:D_SOD-323, symbol Device:D
- C13, C14: LCSC 0402 -> C15195
- J2: LCSC (none) -> C132563; MPN C132563 -> (none)
- R11, R13: LCSC 0603 -> C22813
Connections:
- net BATTERY+: now also D12.1 (K)
- net GND: now also D12.2 (A)
Other:
- moved on the sheet: C21, D10, J7
